Commit message: first step done

File: jackal_package_for_gazebo/urdf/jackal.urdf.xacro (robot description, xacro)
@@ -118,5 +118,5 @@
         <mesh filename="package://jackal_package_for_gazebo/meshes/jackal-base.stl"/>
       </geometry>
-      <material name="dark_grey" />
+      <material name="dark_g3rey" />
     </visual>
     <collision>
@@ -145,5 +145,5 @@
     </visual>
   </link>
-  <joint name="front_fender_joint" type="fixed">
+  <joint name="front_fender_3joint" type="fixed">
     <origin xyz="0 0 0" rpy="0 0 0"/>
     <parent link="chassis_link" />
@@ -216,14 +216,14 @@
   </gazebo>
 <!-- UWB plugin -->
-<!--  <gazebo>-->
-<!--    <plugin name='libgtec_uwb_plugin' filename='libgtec_uwb_plugin.so'>-->
-<!--      <update_rate>25</update_rate>-->
-<!--      <nlosSoftWallWidth>0.25</nlosSoftWallWidth>-->
-<!--      <tag_z_offset>0.3</tag_z_offset>-->
-<!--      <tag_link>base_link</tag_link>-->
-<!--      <anchor_prefix>jackal</anchor_prefix>-->
-<!--      <all_los>false</all_los>-->
-<!--      <tag_id>1</tag_id>-->
-<!--    </plugin>-->
-<!--  </gazebo>-->
+  <gazebo>
+    <plugin name='libgtec_uwb_plugin' filename='libgtec_uwb_plugin.so'>
+      <update_rate>25</update_rate>
+      <nlosSoftWallWidth>0.25</nlosSoftWallWidth>
+      <tag_z_offset>0.3</tag_z_offset>
+      <tag_link>base_link</tag_link>
+      <anchor_prefix>iris</anchor_prefix>
+      <all_los>false</all_los>
+      <tag_id>1</tag_id>
+    </plugin>
+  </gazebo>
 </robot>

Commit message: uwb kalman done

File: jackal_package_for_gazebo/urdf/jackal.urdf.xacro (robot description, xacro)
@@ -224,4 +224,15 @@
   </gazebo>
 <!-- UWB plugin -->
+  <link name="uwb_link">
+    <inertial>
+      <mass value="0.001"/>
+      <origin xyz="0 0 0.2" rpy="0 0 0"/>
+      <inertia ixx="${dummy_inertia}" ixy="0.0" ixz="0.0" iyy="${dummy_inertia}" iyz="0.0" izz="${dummy_inertia}"/>
+    </inertial>
+  </link>
+  <joint name="uwb_joint" type="fixed">
+    <parent link="chassis_link" />
+    <child link="uwb_link" />
+  </joint>
   <gazebo>
     <plugin name='libgtec_uwb_plugin' filename='libgtec_uwb_plugin.so'>
@@ -229,5 +240,5 @@
       <nlosSoftWallWidth>0.25</nlosSoftWallWidth>
       <tag_z_offset>0.3</tag_z_offset>
-      <tag_link>base_link</tag_link>
+      <tag_link>uwb_link</tag_link>
       <anchor_prefix>iris</anchor_prefix>
       <all_los>false</all_los>
